File: dragster/kicad/MontiMiniPcbA/MontiMiniPcbA/MontiMiniPcbA.kicad_pcb (KiCad board)
At the start: 2 copper layers, 45 x 52 mm, 21 parts, among them J1 Power, J2 Serial, J3 Sensors, J4 MotorA, J5 MotorB, SW1 SW_Push, SW2 SW_Push, SW3 ON-OFF, U1 DFROBOT_HR8833, U2 AP1117-33

Commit message: Snapshot 2
Parts:
- J1: footprint Connector_JST:JST_PH_B2B-PH-K_1x02_P2.00mm_Vertical -> Connector_Molex:Molex_KK-254_AE-6410-02A_1x02_P2.54mm_Vertical
- REFH2: moved to B.Cu
- SW3: moved to F.Cu
- moved U2 2.22 mm to (112.5, 85.8)
- moved SW1 1.31 mm to (112.0, 83.8)
- moved SW2 1.31 mm to (112.0, 89.8)
- moved C1 1.22 mm to (110.5, 92.8)
- moved C3 1.22 mm to (115.0, 92.8)
- moved J2 1.22 mm to (142.5, 100.8)
- moved J3 1.22 mm to (119.0, 89.6)
- moved JP1 1.22 mm to (144.0, 85.8)
- moved RZ1 1.22 mm to (121.7, 78.8)
- moved D1 1.00 mm to (109.7, 96.0)
- moved D2 1.00 mm to (148.2, 96.0)
- moved R3 1.00 mm to (114.5, 96.0)
- moved J5 0.88 mm to (146.4, 122.9)
- moved R1 0.50 mm to (147.5, 82.0)
- moved J4 0.46 mm to (119.8, 122.5)
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Routing:
- net +BATT: track 115.6 -> 108.1 mm, vias 0 -> 3
- net GND: track 24.5 -> 30.3 mm, vias 10 -> 12
- net GP9: track 38.9 -> 43.1 mm
- net GP8: track 34.3 -> 38.0 mm
- net Net-(J1-Pad1): track 28.8 -> 31.8 mm, vias 0 -> 1
- net GP2: track 35.8 -> 38.5 mm
- net GP3: track 38.1 -> 40.7 mm
- net GP4: track 25.7 -> 27.0 mm
- net GP7: track 22.2 -> 23.4 mm
- net GP6: track 21.8 -> 23.1 mm
- net GP5: track 23.1 -> 24.2 mm
- net GP12: track 12.8 -> 12.3 mm
- net GP13: track 10.5 -> 9.98 mm
- added copper zone on B.Cu, net +3V3
Other:
- board size 45 x 52 mm -> 45 x 53 mm
