File: dragster/kicad/MontiMiniPcbA/MontiMiniPcbA/MontiMiniPcbA.kicad_sch (KiCad schematic)
At the start: 18 parts, among them J1 Power, J2 Serial, J3 Sensors, J4 MotorA, J5 MotorB, U1 DFROBOT_HR8833

Commit message: Snapshot 2
Parts:
- C1, C3: value (none) -> 4.7uF; footprint (none) -> Capacitor_SMD:C_0805_2012Metric_Pad1.18x1.45mm_HandSolder
- JP1: value (none) -> Bat-Direct; footprint (none) -> Jumper:SolderJumper-2_P1.3mm_Open_Pad1.0x1.5mm
- R1, R3: value (none) -> 220R; footprint (none) -> Resistor_SMD:R_0805_2012Metric_Pad1.20x1.40mm_HandSolder
- SW1, SW2: value (none) -> SW_Push
- SW3: value (none) -> ON-OFF; footprint (none) -> Button_Switch_SMD:SW_SPDT_PCM12
- U2: value (none) -> AP1117-33; footprint (none) -> Package_TO_SOT_SMD:SOT-223-3_TabPin2
Changed lines of the file:
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@@
     (in_bom yes) (on_board yes) (fields_autoplaced)
     (property "Reference" "SW3" (id 0) (at 125.73 22.86 0))
-    (property "Value" "" (id 1) (at 125.73 25.4 0))
-    (property "Footprint" "" (id 2) (at 125.73 29.21 0)
+    (property "Value" "ON-OFF" (id 1) (at 125.73 25.4 0))
+    (property "Footprint" "Button_Switch_SMD:SW_SPDT_PCM12" (id 2) (at 125.73 29.21 0)
       (effects (font (size 1.27 1.27)) hide)
     )
@@
       (effects (font (size 1.27 1.27)) hide)
     )
-    (property "Value" "" (id 1) (at 133.35 54.61 0))
+    (property "Value" "PWR_FLAG" (id 1) (at 133.35 54.61 0))
     (property "Footprint" "" (id 2) (at 133.35 59.69 0)
       (effects (font (size 1.27 1.27)) hide)
@@
     (in_bom yes) (on_board yes) (fields_autoplaced)
     (property "Reference" "SW2" (id 0) (at 213.36 91.44 0))
-    (property "Value" "" (id 1) (at 213.36 91.44 0)
+    (property "Value" "SW_Push" (id 1) (at 213.36 91.44 0)
       (effects (font (size 1.27 1.27)) hide)
     )
@@
     (in_bom yes) (on_board yes) (fields_autoplaced)
     (property "Reference" "U2" (id 0) (at 151.13 21.59 0))
-    (property "Value" "" (id 1) (at 151.13 24.13 0))
-    (property "Footprint" "" (id 2) (at 151.13 24.13 0)
+    (property "Value" "AP1117-33" (id 1) (at 151.13 24.13 0))
+    (property "Footprint" "Package_TO_SOT_SMD:SOT-223-3_TabPin2" (id 2) (at 151.13 24.13 0)
       (effects (font (size 1.27 1.27)) hide)
     )
@@
       (effects (font (size 1.27 1.27)) hide)
     )
-    (property "Value" "" (id 1) (at 151.13 45.72 0))
+    (property "Value" "GND" (id 1) (at 151.13 45.72 0))
     (property "Footprint" "" (id 2) (at 151.13 40.64 0)
       (effects (font (size 1.27 1.27)) hide)
@@
     (in_bom yes) (on_board yes) (fields_autoplaced)
     (property "Reference" "JP1" (id 0) (at 124.46 53.34 0))
-    (property "Value" "" (id 1) (at 124.46 55.88 0))
-    (property "Footprint" "" (id 2) (at 124.46 59.69 0)
+    (property "Value" "Bat-Direct" (id 1) (at 124.46 55.88 0))
+    (property "Footprint" "Jumper:SolderJumper-2_P1.3mm_Open_Pad1.0x1.5mm" (id 2) (at 124.46 59.69 0)
       (effects (font (size 1.27 1.27)) hide)
     )
@@
     (in_bom yes) (on_board yes)
     (property "Reference" "R1" (id 0) (at 213.36 114.3 90))
-    (property "Value" "" (id 1) (at 213.36 116.84 90))
-    (property "Footprint" "" (id 2) (at 213.36 113.538 90)
+    (property "Value" "220R" (id 1) (at 213.36 116.84 90))
+    (property "Footprint" "Resistor_SMD:R_0805_2012Metric_Pad1.20x1.40mm_HandSolder" (id 2) (at 213.36 113.538 90)
       (effects (font (size 1.27 1.27)) hide)
     )
@@
     (in_bom yes) (on_board yes) (fields_autoplaced)
     (property "Reference" "SW1" (id 0) (at 213.36 80.01 0))
-    (property "Value" "" (id 1) (at 213.36 80.01 0)
+    (property "Value" "SW_Push" (id 1) (at 213.36 80.01 0)
       (effects (font (size 1.27 1.27)) hide)
     )
@@
       (effects (font (size 1.27 1.27)) (justify left))
     )
-    (property "Value" "" (id 1) (at 138.43 37.2109 0)
-      (effects (font (size 1.27 1.27)) (justify left))
-    )
-    (property "Footprint" "" (id 2) (at 135.5852 40.64 0)
+    (property "Value" "4.7uF" (id 1) (at 138.43 37.2109 0)
+      (effects (font (size 1.27 1.27)) (justify left))
+    )
+    (property "Footprint" "Capacitor_SMD:C_0805_2012Metric_Pad1.18x1.45mm_HandSolder" (id 2) (at 135.5852 40.64 0)
       (effects (font (size 1.27 1.27)) hide)
     )
@@
     (in_bom yes) (on_board yes)
     (property "Reference" "R3" (id 0) (at 213.36 124.46 90))
-    (property "Value" "" (id 1) (at 213.36 127 90))
-    (property "Footprint" "" (id 2) (at 213.36 123.698 90)
+    (property "Value" "220R" (id 1) (at 213.36 127 90))
+    (property "Footprint" "Resistor_SMD:R_0805_2012Metric_Pad1.20x1.40mm_HandSolder" (id 2) (at 213.36 123.698 90)
       (effects (font (size 1.27 1.27)) hide)
     )
@@
       (effects (font (size 1.27 1.27)) (justify left))
     )
-    (property "Value" "" (id 1) (at 166.37 37.2109 0)
-      (effects (font (size 1.27 1.27)) (justify left))
-    )
-    (property "Footprint" "" (id 2) (at 163.5252 40.64 0)
+    (property "Value" "4.7uF" (id 1) (at 166.37 37.2109 0)
+      (effects (font (size 1.27 1.27)) (justify left))
+    )
+    (property "Footprint" "Capacitor_SMD:C_0805_2012Metric_Pad1.18x1.45mm_HandSolder" (id 2) (at 163.5252 40.64 0)
       (effects (font (size 1.27 1.27)) hide)
     )
@@
     )
     (path "/5ab31f1b-d4d9-453c-be1b-2bb1869af1ae"
-      (reference "J1") (unit 1) (value "Power") (footprint "Connector_JST:JST_PH_B2B-PH-K_1x02_P2.00mm_Vertical")
+      (reference "J1") (unit 1) (value "Power") (footprint "Connector_Molex:Molex_KK-254_AE-6410-02A_1x02_P2.54mm_Vertical")
     )
     (path "/166160b5-b41e-4c78-97fc-65f247e393f9"
