File: dragster/kicad/MontiMiniPcbA/MontiMiniPcbS/MontiMiniPcbS.kicad_pcb (KiCad board)
At the start: 2 copper layers, 45 x 52 mm, 32 parts, among them J1 Sensors, Q1 SFH309, Q2 SFH309, Q3 SFH309, Q4 SFH309, Q5 DMG1012T, Q6 DMG1012T

Commit message: Snapshot 2
Parts:
- moved Q5 1.00 mm to (148.5, 105.5)
- moved Q6 1.00 mm to (133.0, 105.5), turned to 0 degrees
Routing:
- net GND: track 26.3 -> 35.6 mm
- net Net-(D1-Pad1): track 95.3 -> 89.9 mm
- net Net-(Q6-Pad1): track 5.13 -> 7.30 mm
- net Net-(D2-Pad1): track 33.8 -> 32.8 mm
- net Net-(C2-Pad1): track 106.4 -> 105.8 mm
- net A0: track 35.5 -> 36.1 mm
- net GNDREF: vias 8 -> 9

Commit message: Final tweaks
Other:
- board size 45 x 52 mm -> 45 x 53 mm
Changed lines of the file:
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@@
     (property "Sheetname" "")
     (attr smd)
-    (fp_text reference "C1" (at 4.5 -3.5) (layer "F.SilkS")
+    (fp_text reference "C1" (at 4.5 -3) (layer "F.SilkS")
       (effects (font (size 1 1) (thickness 0.15)))
     )
@@
     (property "Sheetname" "")
     (attr smd)
-    (fp_text reference "R8" (at -2.5 -1.65 90) (layer "F.SilkS")
+    (fp_text reference "R8" (at -0.5 -1.5 90) (layer "F.SilkS")
       (effects (font (size 1 1) (thickness 0.15)))
     )
@@
     (property "Sheetname" "")
     (attr smd)
-    (fp_text reference "C2" (at 4.5 3.5) (layer "F.SilkS")
+    (fp_text reference "C2" (at 4.5 3) (layer "F.SilkS")
       (effects (font (size 1 1) (thickness 0.15)))
     )
@@
     (property "Sheetname" "")
     (attr smd)
-    (fp_text reference "R4" (at 1.5 1.65) (layer "B.SilkS")
-      (effects (font (size 1 1) (thickness 0.15)) (justify mirror))
-    )
-    (fp_text value "10k" (at 0 -1.65) (layer "B.Fab")
+    (fp_text reference "R4" (at 0 -1.5) (layer "B.SilkS")
+      (effects (font (size 1 1) (thickness 0.15)) (justify mirror))
+    )
+    (fp_text value "10k" (at 0 1.5) (layer "B.Fab")
       (effects (font (size 1 1) (thickness 0.15)) (justify mirror))
     )
@@
     (property "Sheetname" "")
     (attr smd)
-    (fp_text reference "Q6" (at 0 2) (layer "B.SilkS")
-      (effects (font (size 1 1) (thickness 0.15)) (justify mirror))
-    )
-    (fp_text value "DMG1012T" (at 0 -2.05) (layer "B.Fab")
+    (fp_text reference "Q6" (at -3.5 0) (layer "B.SilkS")
+      (effects (font (size 1 1) (thickness 0.15)) (justify mirror))
+    )
+    (fp_text value "DMG1012T" (at -0.175 2) (layer "B.Fab")
       (effects (font (size 1 1) (thickness 0.15)) (justify mirror))
     )
@@
     (property "Sheetname" "")
     (attr smd)
-    (fp_text reference "R1" (at -3 0) (layer "B.SilkS")
-      (effects (font (size 1 1) (thickness 0.15)) (justify mirror))
-    )
-    (fp_text value "1k" (at 0 -1.65) (layer "B.Fab")
+    (fp_text reference "R1" (at 0 -1.5) (layer "B.SilkS")
+      (effects (font (size 1 1) (thickness 0.15)) (justify mirror))
+    )
+    (fp_text value "1k" (at 0 1.5) (layer "B.Fab")
       (effects (font (size 1 1) (thickness 0.15)) (justify mirror))
     )
@@
       (xy 155.5 110)
       (xy 155.5 105)
-      (xy 155.5 105)
-      (xy 155.5 93)
       (xy 155.5 93)
       (xy 155.5 88)
       (xy 163.5 88)
       (xy 163.5 73)
-      (xy 158.5 68)
-      (xy 123.5 68)
+      (xy 157.5 67)
+      (xy 124.5 67)
       (xy 118.5 73)
       (xy 118.5 88)
       (xy 126.5 88)
       (xy 126.5 93)
-      (xy 126.5 93)
-      (xy 126.5 105)
       (xy 126.5 105)
       (xy 126.5 110)
@@
         (xy 119 87.5)
         (xy 119 73.5)
-        (xy 124 68.5)
-        (xy 158 68.5)
+        (xy 125 67.5)
+        (xy 157 67.5)
       )
     )
