File: dragster/kicad/MontiMiniPcbA/MontiMiniPcbS/MontiMiniPcbS.kicad_pcb (KiCad board)
At the start: 2 copper layers, 45 x 53 mm, 32 parts, among them J1 Sensors, Q1 SFH309, Q2 SFH309, Q3 SFH309, Q4 SFH309, Q5 DMG1012T, Q6 DMG1012T

Commit message: Initial fixes
Parts:
- added REFH1: MountingHole_2.2mm_M2, MountingHole:MountingHole_2.2mm_M2, F.Cu at (141.0, 70.5)
- D1, D2, D3, D4: footprint LED_THT:LED_D3.0mm_Horizontal_O1.27mm_Z2.0mm -> LED_THT:LED_D5.0mm_Horizontal_O1.27mm_Z3.0mm
- moved R3 4.50 mm to (120.0, 84.5)
- moved R8 3.50 mm to (162.0, 83.5)
- moved R1 3.00 mm to (148.0, 99.0)
- moved R2 3.00 mm to (135.0, 99.0)
- moved R4 3.00 mm to (152.0, 99.0)
- moved R5 3.00 mm to (131.0, 99.0)
- moved Q5 2.55 mm to (149.0, 103.0)
- moved Q6 2.55 mm to (133.5, 103.0)
- moved Q4 1.56 mm to (159.4, 80.7)
- moved Q1 1.44 mm to (121.5, 78.5)
- moved J1 1.28 mm to (130.0, 78.5)
- moved Q2 1.03 mm to (133.1, 84.8), turned to 10 degrees
- moved Q3 0.94 mm to (147.6, 84.4), turned to -10 degrees
- moved R7 0.50 mm to (145.0, 89.5)
- moved D2 0.36 mm to (140.0, 86.0), turned to -170 degrees
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Routing:
- net A1: track 30.9 -> 25.5 mm
- net Net-(D1-Pad2): track 6.11 -> 10.6 mm
- net Net-(D1-Pad1): track 89.9 -> 85.9 mm
- net Net-(D4-Pad2): track 3.69 -> 7.65 mm
- net GNDREF: track 8.42 -> 12.0 mm
- net GP14: track 31.1 -> 27.7 mm
- net A3: track 7.51 -> 9.40 mm
- net Net-(C2-Pad1): track 105.8 -> 104.0 mm
- net GP15: track 18.4 -> 16.6 mm
- net Net-(D2-Pad1): track 32.8 -> 31.5 mm
- net VCC: track 59.0 -> 60.2 mm
- net A2: track 8.77 -> 10.0 mm
- net +3V3: track 62.2 -> 63.3 mm
- net Net-(C1-Pad1): track 40.8 -> 39.9 mm
- net Net-(Q6-Pad1): track 7.30 -> 8.01 mm
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