File: dragster/kicad/MontiMiniPcbA/MontiMiniPcbS/MontiMiniPcbS.kicad_sch (KiCad schematic)
At the start: 28 parts, among them Q1 SFH309, Q2 SFH309, Q3 SFH309, Q4 SFH309, Q6 DMG1012T

Commit message: Initial fixes
Parts:
- C1, C2: footprint (none) -> Capacitor_SMD:CP_Elec_6.3x5.9
- C3: value (none) -> 100nF; footprint (none) -> Capacitor_SMD:C_0805_2012Metric_Pad1.18x1.45mm_HandSolder
- D1, D2, D3, D4: value (none) -> TLCR5800
- J1: value (none) -> Sensors; footprint (none) -> Connector_PinHeader_1.27mm:PinHeader_1x10_P1.27mm_Vertical
- Q1, Q2, Q3, Q4: footprint (none) -> LED_THT:LED_D3.0mm_Horizontal_O1.27mm_Z2.0mm
- Q5: value (none) -> DMG1012T; footprint (none) -> Package_TO_SOT_SMD:SOT-323_SC-70_Handsoldering
- Q6: footprint (none) -> Package_TO_SOT_SMD:SOT-323_SC-70_Handsoldering
- R1: value (none) -> 1k; footprint (none) -> Resistor_SMD:R_0805_2012Metric_Pad1.20x1.40mm_HandSolder
- R10, R9: value (none) -> 56R; footprint (none) -> Resistor_SMD:R_0805_2012Metric_Pad1.20x1.40mm_HandSolder
- R11, R12, R13, R14, R2, R4, R5: footprint (none) -> Resistor_SMD:R_0805_2012Metric_Pad1.20x1.40mm_HandSolder
- R3, R6, R7, R8: value (none) -> 7R2; footprint (none) -> Resistor_SMD:R_0805_2012Metric_Pad1.20x1.40mm_HandSolder
