File: monty-half/KiCad/HalfMonti-MainPcbA/HalfMonti-MainPcbA.kicad_pcb (KiCad board)
At the start: 2 copper layers, 45 x 53 mm, 26 parts, among them J1 Power, J2 Serial, J3 Sensors, J4 MotorA, J5 MotorB, SW1 SW_Push, SW2 SW_Push, SW3 ON-OFF, U1 DRV8833PW, U2 AP1117-33

Commit message: Final updates for v2.0 of boards & export
Parts:
- moved J5 0.38 mm to (143.0, 119.4)
Routing:
- net GND: track 31.6 -> 32.7 mm
