File: monty-half/KiCad/HalfMonti-SensorPcbS/HalfMonti-SensorPcbS.kicad_pcb (KiCad board)
At the start: 2 copper layers, 45 x 53 mm, 33 parts, among them J1 Sensors, Q1 SFH309, Q2 SFH309, Q3 SFH309, Q4 SFH309, Q5 DMG1012T, Q6 DMG1012T

Commit message: Update component values on PCBs. Fix PCB labelling R2/R5 issue.
Changed lines of the file:
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@@
     (property "Sheetname" "")
     (attr smd)
-    (fp_text reference "R5" (at -2.46779 -2.49269 180) (layer "F.SilkS")
+    (fp_text reference "R5" (at -2.413 0 180) (layer "F.SilkS")
       (effects (font (size 1 1) (thickness 0.15)))
     )
@@
     (property "Sheetname" "")
     (attr smd)
-    (fp_text reference "R2" (at 2.450358 -2.540001 180) (layer "F.SilkS")
-      (effects (font (size 1 1) (thickness 0.15)))
-    )
+    (fp_text reference "R2" (at 2.413 -0.127 180) (layer "F.SilkS")
+      (effects (font (size 1 1) (thickness 0.15)))
+    )
