File: monty-half/KiCad/HalfMonti-SensorPcbS/HalfMonti-SensorPcbS.kicad_sch (KiCad schematic)
At the start: 28 parts, among them J1 Sensors, Q1 SFH309, Q2 SFH309, Q3 SFH309, Q4 SFH309, Q5 DMG1012T, Q6 DMG1012T

Commit message: Update component values on PCBs. Fix PCB labelling R2/R5 issue.
Parts:
- D1, D2, D3, D4: footprint (none) -> LED_THT:LED_D5.0mm_Horizontal_O1.27mm_Z3.0mm
- Q1, Q2, Q3, Q4: value SFH309 -> BPW85C
- R10, R9: value 56R -> 47R
- R11, R12, R13, R14: value 1.5k -> 2k2
- R3, R6, R7, R8: value 7R2 -> 10R
Changed lines of the file:
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@@
       (effects (font (size 1.27 1.27)) (justify left))
     )
-    (property "Value" "SFH309" (id 1) (at 182.88 71.6406 0)
+    (property "Value" "BPW85C" (id 1) (at 182.88 71.6406 0)
       (effects (font (size 1.27 1.27)) (justify left))
     )
@@
     (property "Reference" "D1" (id 0) (at 62.23 152.4 0))
     (property "Value" "TLCR5800" (id 1) (at 67.31 152.4 0))
-    (property "Footprint" "" (id 2) (at 64.77 152.4 0)
+    (property "Footprint" "LED_THT:LED_D5.0mm_Horizontal_O1.27mm_Z3.0mm" (id 2) (at 64.77 152.4 0)
       (effects (font (size 1.27 1.27)) hide)
     )
@@
       (effects (font (size 1.27 1.27)) (justify left))
     )
-    (property "Value" "SFH309" (id 1) (at 200.66 71.6406 0)
+    (property "Value" "BPW85C" (id 1) (at 200.66 71.6406 0)
       (effects (font (size 1.27 1.27)) (justify left))
     )
@@
       (effects (font (size 1.27 1.27)) (justify right))
     )
-    (property "Value" "1.5k" (id 1) (at 182.88 88.8999 0)
+    (property "Value" "2k2" (id 1) (at 182.88 88.8999 0)
       (effects (font (size 1.27 1.27)) (justify right))
     )
@@
       (effects (font (size 1.27 1.27)) (justify left))
     )
-    (property "Value" "7R2" (id 1) (at 67.31 144.7799 0)
+    (property "Value" "10R" (id 1) (at 67.31 144.7799 0)
       (effects (font (size 1.27 1.27)) (justify left))
     )
@@
       (effects (font (size 1.27 1.27)) (justify left))
     )
-    (property "Value" "SFH309" (id 1) (at 219.71 71.6406 0)
+    (property "Value" "BPW85C" (id 1) (at 219.71 71.6406 0)
       (effects (font (size 1.27 1.27)) (justify left))
     )
@@
     (property "Reference" "D2" (id 0) (at 72.39 85.09 0))
     (property "Value" "TLCR5800" (id 1) (at 77.47 85.09 0))
-    (property "Footprint" "" (id 2) (at 74.93 85.09 0)
+    (property "Footprint" "LED_THT:LED_D5.0mm_Horizontal_O1.27mm_Z3.0mm" (id 2) (at 74.93 85.09 0)
       (effects (font (size 1.27 1.27)) hide)
     )
@@
       (effects (font (size 1.27 1.27)) (justify right))
     )
-    (property "Value" "1.5k" (id 1) (at 200.66 88.8999 0)
+    (property "Value" "2k2" (id 1) (at 200.66 88.8999 0)
       (effects (font (size 1.27 1.27)) (justify right))
     )
@@
       (effects (font (size 1.27 1.27)) (justify left))
     )
-    (property "Value" "SFH309" (id 1) (at 236.22 71.6406 0)
+    (property "Value" "BPW85C" (id 1) (at 236.22 71.6406 0)
       (effects (font (size 1.27 1.27)) (justify left))
     )
@@
       (effects (font (size 1.27 1.27)) (justify left))
     )
-    (property "Value" "7R2" (id 1) (at 87.63 77.4699 0)
+    (property "Value" "10R" (id 1) (at 87.63 77.4699 0)
       (effects (font (size 1.27 1.27)) (justify left))
     )
@@
     (property "Reference" "D4" (id 0) (at 93.98 152.4 0))
     (property "Value" "TLCR5800" (id 1) (at 99.06 152.4 0))
-    (property "Footprint" "" (id 2) (at 96.52 152.4 0)
+    (property "Footprint" "LED_THT:LED_D5.0mm_Horizontal_O1.27mm_Z3.0mm" (id 2) (at 96.52 152.4 0)
       (effects (font (size 1.27 1.27)) hide)
     )
@@
       (effects (font (size 1.27 1.27)) (justify left))
     )
-    (property "Value" "7R2" (id 1) (at 99.06 144.7799 0)
+    (property "Value" "10R" (id 1) (at 99.06 144.7799 0)
       (effects (font (size 1.27 1.27)) (justify left))
     )
@@
       (effects (font (size 1.27 1.27)) (justify left))
     )
-    (property "Value" "7R2" (id 1) (at 77.47 77.4699 0)
+    (property "Value" "10R" (id 1) (at 77.47 77.4699 0)
       (effects (font (size 1.27 1.27)) (justify left))
     )
@@
       (effects (font (size 1.27 1.27)) (justify right))
     )
-    (property "Value" "1.5k" (id 1) (at 219.71 88.8999 0)
+    (property "Value" "2k2" (id 1) (at 219.71 88.8999 0)
       (effects (font (size 1.27 1.27)) (justify right))
     )
@@
     (property "Reference" "D3" (id 0) (at 82.55 85.09 0))
     (property "Value" "TLCR5800" (id 1) (at 87.63 85.09 0))
-    (property "Footprint" "" (id 2) (at 85.09 85.09 0)
+    (property "Footprint" "LED_THT:LED_D5.0mm_Horizontal_O1.27mm_Z3.0mm" (id 2) (at 85.09 85.09 0)
       (effects (font (size 1.27 1.27)) hide)
     )
@@
       (effects (font (size 1.27 1.27)) (justify right))
     )
-    (property "Value" "1.5k" (id 1) (at 236.22 88.8999 0)
+    (property "Value" "2k2" (id 1) (at 236.22 88.8999 0)
       (effects (font (size 1.27 1.27)) (justify right))
     )
@@
       (effects (font (size 1.27 1.27)) (justify left))
     )
-    (property "Value" "56R" (id 1) (at 111.76 135.8899 0)
+    (property "Value" "47R" (id 1) (at 111.76 135.8899 0)
       (effects (font (size 1.27 1.27)) (justify left))
     )
@@
       (effects (font (size 1.27 1.27)) (justify left))
     )
-    (property "Value" "56R" (id 1) (at 110.49 68.5799 0)
+    (property "Value" "47R" (id 1) (at 110.49 68.5799 0)
       (effects (font (size 1.27 1.27)) (justify left))
     )
@@
     )
     (path "/24fd922c-d488-4d61-b6dc-9d3e359ccc82"
-      (reference "Q1") (unit 1) (value "SFH309") (footprint "LED_THT:LED_D3.0mm_Horizontal_O1.27mm_Z2.0mm")
+      (reference "Q1") (unit 1) (value "BPW85C") (footprint "LED_THT:LED_D3.0mm_Horizontal_O1.27mm_Z2.0mm")
     )
     (path "/3e011a46-81bd-4ecd-b93e-57dffb1143e5"
-      (reference "Q2") (unit 1) (value "SFH309") (footprint "LED_THT:LED_D3.0mm_Horizontal_O1.27mm_Z2.0mm")
+      (reference "Q2") (unit 1) (value "BPW85C") (footprint "LED_THT:LED_D3.0mm_Horizontal_O1.27mm_Z2.0mm")
     )
     (path "/47957453-fce7-4d98-833c-e34bb8a852a5"
-      (reference "Q3") (unit 1) (value "SFH309") (footprint "LED_THT:LED_D3.0mm_Horizontal_O1.27mm_Z2.0mm")
+      (reference "Q3") (unit 1) (value "BPW85C") (footprint "LED_THT:LED_D3.0mm_Horizontal_O1.27mm_Z2.0mm")
     )
     (path "/a8a389df-8d18-4e17-a74f-f60d5d77371e"
-      (reference "Q4") (unit 1) (value "SFH309") (footprint "LED_THT:LED_D3.0mm_Horizontal_O1.27mm_Z2.0mm")
+      (reference "Q4") (unit 1) (value "BPW85C") (footprint "LED_THT:LED_D3.0mm_Horizontal_O1.27mm_Z2.0mm")
     )
     (path "/9c6b6a16-9b62-44e4-a22e-f145da2ae51d"
@@
     )
     (path "/46c1d222-181e-47b5-9380-eaf9d6e17a22"
-      (reference "R3") (unit 1) (value "7R2") (footprint "Resistor_SMD:R_0805_2012Metric_Pad1.20x1.40mm_HandSolder")
+      (reference "R3") (unit 1) (value "10R") (footprint "Resistor_SMD:R_0805_2012Metric_Pad1.20x1.40mm_HandSolder")
     )
     (path "/df5c9f6b-a62e-44ba-997f-b2cf3279c7d4"
@@
     )
     (path "/c9badf80-21f8-404a-b5df-18e98bffebf9"
-      (reference "R6") (unit 1) (value "7R2") (footprint "Resistor_SMD:R_0805_2012Metric_Pad1.20x1.40mm_HandSolder")
+      (reference "R6") (unit 1) (value "10R") (footprint "Resistor_SMD:R_0805_2012Metric_Pad1.20x1.40mm_HandSolder")
     )
     (path "/b8e1a8b8-63f0-4e53-a6cb-c8edf9a649c4"
-      (reference "R7") (unit 1) (value "7R2") (footprint "Resistor_SMD:R_0805_2012Metric_Pad1.20x1.40mm_HandSolder")
+      (reference "R7") (unit 1) (value "10R") (footprint "Resistor_SMD:R_0805_2012Metric_Pad1.20x1.40mm_HandSolder")
     )
     (path "/befab85e-9093-46eb-b656-c322a425c12f"
-      (reference "R8") (unit 1) (value "7R2") (footprint "Resistor_SMD:R_0805_2012Metric_Pad1.20x1.40mm_HandSolder")
+      (reference "R8") (unit 1) (value "10R") (footprint "Resistor_SMD:R_0805_2012Metric_Pad1.20x1.40mm_HandSolder")
     )
     (path "/f3c1aa2b-1d9c-4e97-856e-19830bade54c"
-      (reference "R9") (unit 1) (value "56R") (footprint "Resistor_SMD:R_0805_2012Metric_Pad1.20x1.40mm_HandSolder")
+      (reference "R9") (unit 1) (value "47R") (footprint "Resistor_SMD:R_0805_2012Metric_Pad1.20x1.40mm_HandSolder")
     )
     (path "/f2ed98ad-ee43-4932-981a-d440169ac48f"
-      (reference "R10") (unit 1) (value "56R") (footprint "Resistor_SMD:R_0805_2012Metric_Pad1.20x1.40mm_HandSolder")
+      (reference "R10") (unit 1) (value "47R") (footprint "Resistor_SMD:R_0805_2012Metric_Pad1.20x1.40mm_HandSolder")
     )
     (path "/3f43c2dc-daa2-45ba-b8ca-7ae5aebed882"
-      (reference "R11") (unit 1) (value "1.5k") (footprint "Resistor_SMD:R_0805_2012Metric_Pad1.20x1.40mm_HandSolder")
+      (reference "R11") (unit 1) (value "2k2") (footprint "Resistor_SMD:R_0805_2012Metric_Pad1.20x1.40mm_HandSolder")
     )
     (path "/97693043-81ba-44a2-b87b-aca6193e0970"
-      (reference "R12") (unit 1) (value "1.5k") (footprint "Resistor_SMD:R_0805_2012Metric_Pad1.20x1.40mm_HandSolder")
+      (reference "R12") (unit 1) (value "2k2") (footprint "Resistor_SMD:R_0805_2012Metric_Pad1.20x1.40mm_HandSolder")
     )
     (path "/dfba7148-cad3-4f40-9835-b1394bd30a2c"
-      (reference "R13") (unit 1) (value "1.5k") (footprint "Resistor_SMD:R_0805_2012Metric_Pad1.20x1.40mm_HandSolder")
+      (reference "R13") (unit 1) (value "2k2") (footprint "Resistor_SMD:R_0805_2012Metric_Pad1.20x1.40mm_HandSolder")
     )
     (path "/f2044410-03ac-4994-9652-9e5f480320f0"
-      (reference "R14") (unit 1) (value "1.5k") (footprint "Resistor_SMD:R_0805_2012Metric_Pad1.20x1.40mm_HandSolder")
-    )
-  )
+      (reference "R14") (unit 1) (value "2k2") (footprint "Resistor_SMD:R_0805_2012Metric_Pad1.20x1.40mm_HandSolder")
+    )
+  )
