File: dragster/kicad/DragNoseV2/DragNoseV2.kicad_pcb (KiCad board)
At the start: 2 copper layers, 112 x 112.2 mm, 44 parts, among them J1 Conn_01x10_Male, Q1 SFH309, Q2 SFH309, Q3 SFH309, Q4 SFH309, Q5 SFH309, Q6 SFH309, Q7 DMG1012T, U1 ITR8307-S17-TR8, U2 ITR8307-S17-TR8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

Commit message: Final tweaks before v2 to JLCPCB manufacture
Parts:
- added REFholerightmf: locked, MountingHole:MountingHole_2.2mm_M2, F.Cu at (101.4, 69.1)
