File: kicad/line-sensor-mini-5/line-sensor-mini-5.kicad_pcb (KiCad board)
At the start: 2 copper layers, 72.4 x 19.7 mm, 28 parts, among them J1 10x0.5mm FPC, Q1 BC817, Q2 DMG1012T, Q3 PT0805CS, Q4 PT0805CS, Q5 PT0805CS, Q6 PT0805CS, Q7 BC817, Q8 DMG1012T

Commit message: Add test code for new 1/2 size line-follower mouse
Routing:
- net Net-(Q1-B): track 6.07 -> 6.60 mm
Changed lines of the file:
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@@
 		(tags "resistor")
 		(property "Reference" "R9"
-			(at 0.123712 -4.10897 -90)
+			(at 0.001517 1.685801 -90)
 			(layer "F.SilkS")
 			(effects
@@
 		(tags "resistor")
 		(property "Reference" "R10"
-			(at 0.019944 -4.087888 90)
+			(at 0 1.905 90)
 			(layer "F.SilkS")
 			(effects
@@
 	)
 	(segment
-		(start 169.2025 100.98)
-		(end 171.085 100.98)
+		(start 171.44 100.83)
+		(end 171.44 103.5325)
 		(width 0.25)
 		(layer "F.Cu")
@@
 	)
 	(segment
-		(start 171.085 103.7625)
+		(start 171.44 103.5325)
 		(end 171.1475 103.825)
 		(width 0.25)
@@
 	)
 	(segment
-		(start 168.275 100.0525)
-		(end 169.2025 100.98)
+		(start 169.0525 100.83)
+		(end 171.44 100.83)
 		(width 0.25)
 		(layer "F.Cu")
@@
 	)
 	(segment
-		(start 171.085 100.98)
-		(end 171.085 103.7625)
+		(start 168.275 100.0525)
+		(end 169.0525 100.83)
 		(width 0.25)
 		(layer "F.Cu")
