File: kicad/half-monty-2/half-monty-2-sensors.kicad_sch (KiCad schematic)
At the start: 29 parts, among them Q1 BC817, Q2 SSM3K122TU, Q3 PT100MF0MP, Q4 PT100MF0MP, Q5 PT100MF0MP, Q6 BC817, Q7 SSM3K122TU, Q8 PT100MF0MP

Commit message: Update component values after prototype assembly
Parts:
- C7: value 100nF -> 2.2uF
- R11, R13: value 2k2 -> 270R
- R15, R8: value 1k5 -> 200R
- R7: value 220R -> 10R
- R9: value 22R -> 20R
Changed lines of the file:
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@@
 			)
 		)
-		(property "Value" "2k2"
+		(property "Value" "270R"
 			(at 175.26 137.1599 0)
 			(effects
@@
 			)
 		)
-		(property "Value" "100nF"
+		(property "Value" "2.2uF"
 			(at 120.65 137.1663 0)
 			(effects
@@
 			)
 		)
-		(property "Value" "1k5"
+		(property "Value" "200R"
 			(at 195.58 137.1599 0)
 			(effects
@@
 			)
 		)
-		(property "Value" "22R"
+		(property "Value" "20R"
 			(at 142.24 38.0999 0)
 			(effects
@@
 		(fields_autoplaced yes)
 		(property "Reference" "R7"
-			(at 120.65 104.14 0)
-			(effects
-				(font
-					(size 1.27 1.27)
-				)
-				(justify left)
-			)
-		)
-		(property "Value" "220R"
-			(at 120.65 106.68 0)
+			(at 120.65 104.1399 0)
+			(effects
+				(font
+					(size 1.27 1.27)
+				)
+				(justify left)
+			)
+		)
+		(property "Value" "10R"
+			(at 120.65 106.6799 0)
 			(effects
 				(font
@@
 			)
 		)
-		(property "Value" "1k5"
+		(property "Value" "200R"
 			(at 134.62 137.1599 0)
 			(effects
@@
 			)
 		)
-		(property "Value" "2k2"
+		(property "Value" "270R"
 			(at 154.94 137.1599 0)
 			(effects
