File: kicad/wall-sens-fpc-4/wall-sens-fpc-4.kicad_sch (KiCad schematic)
At the start: 30 parts, among them J1 10x0.5mm FPC, Q1 PT100MF0MP, Q2 PT100MF0MP, Q3 PT100MF0MP, Q4 PT100MF0MP, Q5 BC817, Q6 SSM3K122TU, Q7 BC817, Q8 SSM3K122TU

Commit message: New version of wall-follower for full size. Add new design Half-Monty-2
Parts:
- C2: value 22uF -> 47uF; footprint Capacitor_SMD:C_0805_2012Metric -> Capacitor_SMD:C_1206_3216Metric
Changed lines of the file:
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@@
 			)
 		)
-		(property "Value" "22uF"
+		(property "Value" "47uF"
 			(at 105.41 62.2362 0)
 			(effects
@@
 			)
 		)
-		(property "Footprint" "Capacitor_SMD:C_0805_2012Metric"
+		(property "Footprint" "Capacitor_SMD:C_1206_3216Metric"
 			(at 102.87 60.96 0)
 			(effects

Commit message: Update component values after prototype assembly
Parts:
- C1: value 100nF -> 2.2uF
- R1, R4: value 1k5 -> 510R
- R12: value 22R -> 20R
- R2, R3: value 2k2 -> 680R
- R8: value 220R -> 15R
Changed lines of the file:
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@@
 			)
 		)
-		(property "Value" "2k2"
+		(property "Value" "680R"
 			(at 154.94 135.8899 0)
 			(effects
@@
 			)
 		)
-		(property "Value" "100nF"
+		(property "Value" "2.2uF"
 			(at 100.33 135.8963 0)
 			(effects
@@
 			)
 		)
-		(property "Value" "1k5"
+		(property "Value" "510R"
 			(at 175.26 135.8899 0)
 			(effects
@@
 			)
 		)
-		(property "Value" "22R"
+		(property "Value" "20R"
 			(at 121.92 36.8299 0)
 			(effects
@@
 		(fields_autoplaced yes)
 		(property "Reference" "R8"
-			(at 100.33 102.87 0)
-			(effects
-				(font
-					(size 1.27 1.27)
-				)
-				(justify left)
-			)
-		)
-		(property "Value" "220R"
-			(at 100.33 105.41 0)
+			(at 100.33 102.8699 0)
+			(effects
+				(font
+					(size 1.27 1.27)
+				)
+				(justify left)
+			)
+		)
+		(property "Value" "15R"
+			(at 100.33 105.4099 0)
 			(effects
 				(font
@@
 			)
 		)
-		(property "Value" "1k5"
+		(property "Value" "510R"
 			(at 114.3 135.8899 0)
 			(effects
@@
 			)
 		)
-		(property "Value" "2k2"
+		(property "Value" "680R"
 			(at 134.62 135.8899 0)
 			(effects
